File: hardware/pcb/wakelight.kicad_pcb (KiCad board)
At the start: 2 copper layers, 55 x 42 mm, 35 parts, among them J1 USB-C 16P, J2 DMX OUT, Q1 SS8050, Q2 SS8050, SW1 EN, SW2 BOOT, U1 ESP32-WROOM-32E-N8, U2 CH340C, U3 AMS1117-3.3, U4 THVD1410DR

Commit message: WakeLight v1.1: PCB-mount Neutrik NC5FAH 5-pin XLR DMX output
Board widened to 66x42mm, XLR footprint verified against the official
Neutrik drilling plan, regulator corner re-placed, DRC clean (0 errors,
0 unconnected). Schematic updated (ERC clean), v1.0 terminal-variant fab
files archived, docs and sourcing updated.

Co-Authored-By: Claude Fable 5 <noreply@anthropic.com>
Parts:
- J2: value DMX OUT -> NC5FAH DMX OUT; footprint TerminalBlock_Phoenix_MKDS-1,5-3-5.08_1x03_P5.08mm_Horizontal -> Jack_XLR_Neutrik_NC5FAH_Horizontal
- moved H3 11.0 mm to (62.5, 38.5)
- moved H4 11.0 mm to (62.5, 3.50)
- moved R6 10.8 mm to (58.2, 36.5)
- moved U3 9.46 mm to (50.5, 37.9), turned to 0 degrees
- moved C2 7.50 mm to (44.8, 37.9)
- moved D1 6.73 mm to (56.5, 36.5)
- moved J2 6.51 mm to (48.9, 17.0), turned to 0 degrees
Routing:
- net +3V3: track 110.5 -> 128.0 mm
- net DMX_B: track 17.7 -> 26.3 mm
- net GND: track 45.2 -> 51.9 mm, vias 24 -> 22
- net RTS: track 36.0 -> 29.8 mm
- net Q_IO0_B: track 7.55 -> 12.6 mm
- net PWR_LED: track 5.19 -> 1.72 mm
- net EN: track 26.4 -> 23.4 mm
- net IO0: track 40.8 -> 38.9 mm, vias 4 -> 3
- net DTR: track 23.6 -> 24.5 mm, vias 2 -> 0
- net DMX_A: track 26.7 -> 27.2 mm, vias 3 -> 2
Other:
- board size 55 x 42 mm -> 66 x 42 mm
- board text added: "DMX OUT"
- board text added: "WakeLight v1.1"
- board text removed: "DMX 1:GND 2:D- 3:D+"
- board text removed: "WakeLight v1.0"
